Commit message: urdf 수정

File: src/sim/urdf/robot.urdf (robot description, URDF)
Before this commit: robot my_robot, 13 links, 12 joints
Links:
- link base: geometry collision mesh filename=package://sim/meshes/base.stl scale=0.001 0.001 0.001; visual mesh filename=package://sim/meshes/base.stl scale=0.001 0.001 0.001
- link joint1: geometry collision mesh filename=package://sim/meshes/joint1.stl scale=0.001 0.001 0.001; visual mesh filename=package://sim/meshes/joint1.stl scale=0.001 0.001 0.001
- link joint2: geometry collision mesh filename=package://sim/meshes/joint2.stl scale=0.001 0.001 0.001; visual mesh filename=package://sim/meshes/joint2.stl scale=0.001 0.001 0.001
- link link1_1: geometry collision mesh filename=package://sim/meshes/link1_1.stl scale=0.001 0.001 0.001; visual mesh filename=package://sim/meshes/link1_1.stl scale=0.001 0.001 0.001
- link link1_2: geometry collision mesh filename=package://sim/meshes/link1_2.stl scale=0.001 0.001 0.001; visual mesh filename=package://sim/meshes/link1_2.stl scale=0.001 0.001 0.001
- link link1_3: geometry collision mesh filename=package://sim/meshes/link1_3.stl scale=0.001 0.001 0.001; visual mesh filename=package://sim/meshes/link1_3.stl scale=0.001 0.001 0.001
- link link2_1: geometry collision mesh filename=package://sim/meshes/link2_1.stl scale=0.001 0.001 0.001; visual mesh filename=package://sim/meshes/link2_1.stl scale=0.001 0.001 0.001
- link link2_2: geometry collision mesh filename=package://sim/meshes/link2_2.stl scale=0.001 0.001 0.001; visual mesh filename=package://sim/meshes/link2_2.stl scale=0.001 0.001 0.001
- link rs02_1: geometry collision mesh filename=package://sim/meshes/RS02(0.0.0).stl scale=0.001 0.001 0.001; visual mesh filename=package://sim/meshes/RS02(0.0.0).stl scale=0.001 0.001 0.001
- link rs02_2: geometry collision mesh filename=package://sim/meshes/RS02(0.0.0).stl scale=0.001 0.001 0.001; visual mesh filename=package://sim/meshes/RS02(0.0.0).stl scale=0.001 0.001 0.001
- link rs02_3: geometry collision mesh filename=package://sim/meshes/RS02(0.0.0).stl scale=0.001 0.001 0.001; visual mesh filename=package://sim/meshes/RS02(0.0.0).stl scale=0.001 0.001 0.001
- link rs03: geometry collision mesh filename=package://sim/meshes/RS03(0.0.0).stl scale=0.001 0.001 0.001; visual mesh filename=package://sim/meshes/RS03(0.0.0).stl scale=0.001 0.001 0.001

Commit message: 축 수정

File: src/sim/urdf/robot.urdf (robot description, URDF)
Before this commit: robot my_robot, 13 links, 12 joints
Joints:
- joint j1: axis 0 0 1 -> 0 0 -1
- joint j2: axis 0 0 1 -> 0 0 -1
- joint j3: axis 0 0 1 -> 0 0 -1
- joint j4: axis 0 0 1 -> 0 0 -1

Commit message: com inertial 수정

File: src/sim/urdf/robot.urdf (robot description, URDF)
Before this commit: robot my_robot, 13 links, 12 joints
Links:
- link base: mass 0.40598 -> 0.398399734
- link joint1: mass 0.28684 -> 0.293398076
- link joint2: mass 0.16391 -> 0.169648237
- link link1_1: mass 0.25495 -> 0.319496008
- link link1_2: mass 0.504 -> 0.508299975
- link link1_3: mass 0.21978 -> 0.279149934
- link link2_1: mass 0.112 -> 0.188800061
- link link2_2: mass 0.111 -> 0.170500037

Commit message: urdf 완

File: src/sim/urdf/robot.urdf (robot description, URDF)
Before this commit: robot my_robot, 13 links, 12 joints
Links:
- link base: mass 0.398399734 -> 0.6248
- link joint1: mass 0.293398076 -> 0.270398
- link joint2: mass 0.169648237 -> 0.151798
- link link1_1: mass 0.319496008 -> 0.236296
- link link2_1: mass 0.188800061 -> 0.112000
- link rs02_1: mass 0.405 -> 0.4116
- link rs02_2: mass 0.405 -> 0.4116
- link rs02_3: mass 0.405 -> 0.4116
- link rs03: mass 0.88 -> 0.9244
Joints:
- joint j1: axis 0 0 -1 -> 0 0 1; origin xyz=0 0 0 rpy=0 0 0 -> xyz=0 0 0 rpy=0 3.1415926 0
- joint j2: axis 0 0 -1 -> 0 0 1; origin xyz=0 0 0 rpy=0 0 0 -> xyz=0 0 0 rpy=3.1415926 0 0
- joint j2_2: origin xyz=0 0.05 0.05715 rpy=-1.5708 0 0 -> xyz=0 0.05 -0.05715 rpy=-1.5708 0 0
- joint j2_3: origin xyz=0 0 0.3 rpy=0 0 0 -> xyz=0 0 0.3 rpy=0 0 3.1415926
- joint j3: axis 0 0 -1 -> 0 0 1; origin xyz=0 0 0 rpy=0 0 0 -> xyz=0 0 0 rpy=3.1415926 0 3.1415926
- joint j4: axis 0 0 -1 -> 0 0 1; origin xyz=0 0 0 rpy=0 0 0 -> xyz=0 0 0 rpy=3.1415926 0 0
- joint j4_2: origin xyz=0 0 0.035 rpy=0 0 0 -> xyz=0 0 0.035 rpy=0 3.1415926 0
- joint m2: origin xyz=0 -0.0637 0.068 rpy=1.5708 0 0 -> xyz=0 -0.0637 -0.068 rpy=1.5708 0 0
- joint m4: origin xyz=0 -0.0502 0.055 rpy=1.5708 0 0 -> xyz=0 -0.0502 -0.055 rpy=1.5708 0 0

Commit message: clamp  제한

File: src/sim/urdf/robot.urdf (robot description, URDF)
Before this commit: robot my_robot, 13 links, 12 joints
Joints:
- joint j2: limit lower=-2.5 upper=2.5 effort=50 velocity=100 -> lower=-1.78 upper=1.78 effort=50 velocity=100

Commit message: 3월 21일 가장 최신

File: src/sim/urdf/robot.urdf (robot description, URDF)
Before this commit: robot my_robot, 13 links, 12 joints
Links:
- removed link joint2
- added link link2_3, mass 0.170500037; collision mesh filename=package://sim/meshes/link2_3.stl scale=0.001 0.001 0.001; visual mesh filename=package://sim/meshes/link2_3.stl scale=0.001 0.001 0.001
- link link2_1: mass 0.112000 -> 0.151798
- link link2_2: mass 0.170500037 -> 0.112000
Joints:
- removed joint j4_2
- removed joint m4
- added joint j3_2: type fixed, parent link2_1, child link2_2, origin xyz=0 -0.050 -0.05315 rpy=1.5708 0 0
- added joint j3_3: type fixed, parent link2_2, child link2_3, origin xyz=0 0 0.23 rpy=0 0 0
- joint ee_fixed: parent link2_2 -> link2_3
- joint j1: origin xyz=0 0 0 rpy=0 3.1415926 0 -> xyz=0 0 0 rpy=3.14159 0 0
- joint j3: child joint2 -> link2_1
- joint j4: child link2_1 -> rs02_3; origin xyz=0 0 0 rpy=3.1415926 0 0 -> xyz=0 -0.06185 0.05 rpy=1.5708 0 0; parent rs02_3 -> link2_3
- joint m1: origin xyz=0 0 0.1015 rpy=0 0 0 -> xyz=0 0 0.1002 rpy=0 0 0
- joint m2: origin xyz=0 -0.0637 -0.068 rpy=1.5708 0 0 -> xyz=-0.0362 0 -0.0893 rpy=1.5708 0 -1.5708
- joint m3: origin xyz=0 0.06585 0.050 rpy=-1.5708 0 0 -> xyz=0 0.06735 0.050 rpy=-1.5708 0 0

Commit message: 6dof urdf 완

File: src/sim/urdf/robot.urdf (robot description, URDF)
Before this commit: robot my_robot, 13 links, 12 joints
Links:
- added link link3_1, mass 0.170500037; collision mesh filename=package://sim/meshes/link3_1.stl scale=0.001 0.001 0.001; visual mesh filename=package://sim/meshes/link3_1.stl scale=0.001 0.001 0.001
- added link link3_2, mass 0.170500037; collision mesh filename=package://sim/meshes/link3_2.stl scale=0.001 0.001 0.001; visual mesh filename=package://sim/meshes/link3_2.stl scale=0.001 0.001 0.001
- added link rs00_1, mass 0.9244; collision mesh filename=package://sim/meshes/RS00.stl scale=0.001 0.001 0.001; visual mesh filename=package://sim/meshes/RS00.stl scale=0.001 0.001 0.001
- added link rs00_2, mass 0.9244; collision mesh filename=package://sim/meshes/RS00.stl scale=0.001 0.001 0.001; visual mesh filename=package://sim/meshes/RS00.stl scale=0.001 0.001 0.001
Joints:
- added joint j5: type revolute, parent rs00_1, child link3_2, origin xyz=0 0 0 rpy=0 3.14159 0, axis 0 0 1, limit lower=-3.14159 upper=3.14159 effort=50 velocity=100
- added joint m4: type fixed, parent link2_3, child rs02_3, origin xyz=0 -0.06585 0.05 rpy=1.5708 0 0, axis 0 0 1, limit lower=-3.14159 upper=3.14159 effort=50 velocity=100
- added joint m5: type fixed, parent link3_1, child rs00_1, origin xyz=0 0.0724 -0.053 rpy=-1.5708 0 0
- added joint m6: type fixed, parent link3_2, child rs00_2, origin xyz=0 0.072 -0.058 rpy=-1.5708 0 0
- joint ee_fixed: axis (none) -> 0 0 1; limit (none) -> lower=-3.14159 upper=3.14159 effort=50 velocity=100; origin xyz=0 0 0.23 rpy=0 0 0 -> xyz=0 0 0 rpy=3.14159 0 0; parent link2_3 -> rs00_2; type fixed -> revolute
- joint j4: child rs02_3 -> link3_1; origin xyz=0 -0.06185 0.05 rpy=1.5708 0 0 -> xyz=0 0 0 rpy=0 3.14159 0; parent link2_3 -> rs02_3

Commit message: Update robot.urdf

File: src/sim/urdf/robot.urdf (robot description, URDF)
Before this commit: robot my_robot, 17 links, 16 joints
Links:
- link rs00_1: mass 0.9244 -> 0.3100
- link rs00_2: mass 0.9244 -> 0.3100

Commit message: 6dof 수정 중

File: src/sim/urdf/robot.urdf (robot description, URDF)
Before this commit: robot my_robot, 17 links, 16 joints
Links:
- removed link ee_link
- added link finger_l, mass 0.1; collision mesh filename=package://sim/meshes/finger_l.stl scale=0.001 0.001 0.001; visual mesh filename=package://sim/meshes/finger_l.stl scale=0.001 0.001 0.001
- added link finger_r, mass 0.1; collision mesh filename=package://sim/meshes/finger_r.stl scale=0.001 0.001 0.001; visual mesh filename=package://sim/meshes/finger_r.stl scale=0.001 0.001 0.001
- added link gripper, mass 0.1; collision mesh filename=package://sim/meshes/gripper.stl scale=0.001 0.001 0.001; visual mesh filename=package://sim/meshes/gripper.stl scale=0.001 0.001 0.001
- added link rs05, mass 0.9244; collision mesh filename=package://sim/meshes/RS05.stl scale=0.001 0.001 0.001; visual mesh filename=package://sim/meshes/RS05.stl scale=0.001 0.001 0.001
Joints:
- removed joint ee_fixed
- added joint finger_l: type prismatic, parent gripper, child finger_l, origin xyz=0 0.07375 -0.0198 rpy=0 0 0, axis 0 -1 0, limit lower=0 upper=0.05 effort=50 velocity=100, mimic joint=finger_r multiplier=1.0 offset=0
- added joint finger_r: type prismatic, parent gripper, child finger_r, origin xyz=0 -0.07375 -0.0198 rpy=0 0 0, axis 0 1 0, limit lower=0 upper=0.05 effort=50 velocity=100
- added joint j6: type revolute, parent rs00_2, child rs05, origin xyz=0 0 0.0500 rpy=0 0 0, axis 0 0 1, limit lower=-3.14159 upper=3.14159 effort=50 velocity=100
- added joint m7: type fixed, parent rs05, child gripper, origin xyz=0 0 0 rpy=0 3.14159 0

Commit message: 6dof_urdf inertial 외 끝

File: src/sim/urdf/robot.urdf (robot description, URDF)
Before this commit: robot my_robot, 20 links, 19 joints
Links:
- added link case, mass 0.1; collision mesh filename=package://sim/meshes/case.stl scale=0.001 0.001 0.001; visual mesh filename=package://sim/meshes/case.stl scale=0.001 0.001 0.001
- added link connect_00, mass 0.1; collision mesh filename=package://sim/meshes/connect_00.stl scale=0.001 0.001 0.001; visual mesh filename=package://sim/meshes/connect_00.stl scale=0.001 0.001 0.001
- added link connect_05, mass 0.1; collision mesh filename=package://sim/meshes/connect_05.stl scale=0.001 0.001 0.001; visual mesh filename=package://sim/meshes/connect_05.stl scale=0.001 0.001 0.001
Joints:
- added joint case: type fixed, parent rs05, child case, origin xyz=0 0 0 rpy=0 0 0
- added joint connect: type fixed, parent connect_00, child connect_05, origin xyz=0 0 -0.02 rpy=3.141592 0 0
- added joint gripper_base: type fixed, parent rs05, child gripper, origin xyz=0 0 0 rpy=0 3.14159 0
- joint finger_l: origin xyz=0 0.07375 -0.0198 rpy=0 0 0 -> xyz=0 0.0625 -0.0198 rpy=0 0 0
- joint finger_r: origin xyz=0 -0.07375 -0.0198 rpy=0 0 0 -> xyz=0 -0.0625 -0.0198 rpy=0 0 0
- joint j3_2: origin xyz=0 -0.050 -0.05315 rpy=1.5708 0 0 -> xyz=0 -0.050 -0.07415 rpy=1.5708 0 0
- joint j6: child rs05 -> connect_00; origin xyz=0 0 0.0500 rpy=0 0 0 -> xyz=0 0 0 rpy=3.141592 0 0
- joint m4: axis 0 0 1 -> (none); limit lower=-3.14159 upper=3.14159 effort=50 velocity=100 -> (none)
- joint m6: origin xyz=0 0.072 -0.058 rpy=-1.5708 0 0 -> xyz=0 0.0724 -0.058 rpy=-1.5708 0 0
- joint m7: child gripper -> rs05; origin xyz=0 0 0 rpy=0 3.14159 0 -> xyz=0 0 0.06 rpy=0 0 0; parent rs05 -> connect_05

Commit message: 이너셜 추가

File: src/sim/urdf/robot.urdf (robot description, URDF)
Before this commit: robot my_robot, 23 links, 22 joints
Links:
- removed link case
- removed link connect_00
- removed link connect_05
- added link link3_3, mass 0.202651; collision mesh filename=package://sim/meshes/link3_3.stl scale=0.001 0.001 0.001; visual mesh filename=package://sim/meshes/link3_3.stl scale=0.001 0.001 0.001
- link base: mass 0.6248 -> 0.685513
- link finger_l: mass 0.1 -> 0.030964
- link finger_r: mass 0.1 -> 0.030964
- link gripper: mass 0.1 -> 0.090928
- link joint1: mass 0.270398 -> 0.431305
- link link1_1: mass 0.236296 -> 0.350100
- link link1_2: mass 0.508299975 -> 0.502204
- link link1_3: mass 0.279149934 -> 0.279601
- link link2_1: mass 0.151798 -> 0.361563
- link link2_2: mass 0.112000 -> 0.154772
- link link2_3: mass 0.170500037 -> 0.302349
- link link3_1: mass 0.170500037 -> 0.264011
- link link3_2: mass 0.170500037 -> 0.259261
- link rs00_1: mass 0.9244 -> 0.311841
- link rs00_2: mass 0.9244 -> 0.311841
- link rs02_1: mass 0.4116 -> 0.411618
- link rs02_2: mass 0.4116 -> 0.411618
- link rs02_3: mass 0.4116 -> 0.411618
- link rs03: mass 0.9244 -> 0.924357
- link rs05: mass 0.9244 -> 0.191090
Joints:
- removed joint case
- removed joint connect
- joint finger_l: origin xyz=0 0.0625 -0.0198 rpy=0 0 0 -> xyz=0 0.06475 -0.0218 rpy=0 0 0
- joint finger_r: limit lower=0 upper=0.05 effort=50 velocity=100 -> lower=0 upper=0.0447 effort=50 velocity=100; origin xyz=0 -0.0625 -0.0198 rpy=0 0 0 -> xyz=0 -0.06475 -0.0218 rpy=0 0 0
- joint j3: origin xyz=0 0 0 rpy=3.1415926 0 3.1415926 -> xyz=0 0 0 rpy=3.1415926 0 0
- joint j6: child connect_00 -> link3_3; origin xyz=0 0 0 rpy=3.141592 0 0 -> xyz=0 0 0 rpy=0 3.141592 3.141592
- joint m7: origin xyz=0 0 0.06 rpy=0 0 0 -> xyz=0 0 -0.093 rpy=0 3.141592 1.570791; parent connect_05 -> link3_3

Commit message: 이너셜 완료

File: src/sim/urdf/robot.urdf (robot description, URDF)
Before this commit: robot my_robot, 21 links, 20 joints
Joints:
- joint m1: origin xyz=0 0 0.1002 rpy=0 0 0 -> xyz=0 0 0.1002 rpy=0 0 1.570796

Commit message: 수정

File: src/sim/urdf/robot.urdf (robot description, URDF)
Before this commit: robot my_robot, 21 links, 20 joints
Joints:
- joint j3_2: origin xyz=0 -0.050 -0.07415 rpy=1.5708 0 0 -> xyz=0 -0.050 -0.07465 rpy=1.5708 0 0

Commit message: plan_node 역할 쪼개기

File: src/sim/urdf/robot.urdf (robot description, URDF)
Before this commit: robot my_robot, 21 links, 20 joints
Links:
- added link cage, mass 1.0; collision mesh filename=package://sim/meshes/Cage.stl scale=0.001 0.001 0.001; visual mesh filename=package://sim/meshes/Cage.stl scale=0.001 0.001 0.001
- link link1_3: mass 0.279601 -> 0.322751
- link link2_1: mass 0.361563 -> 0.697618
- link link2_3: mass 0.302349 -> 0.288847
Joints:
- added joint cage_to_base: type fixed, parent cage, child base, origin xyz=0 0 0.03 rpy=0 0 0

Commit message: Add files via upload

File: src/sim/urdf/robot.urdf (robot description, URDF)
Before this commit: robot my_robot_with_cage, 22 links, 21 joints
Links:
- link link2_1: mass 0.697618 -> 0.840115
- link link2_3: mass 0.288847 -> 0.235762
- link link3_1: mass 0.264011 -> 0.215857
- link link3_2: mass 0.259261 -> 0.202646
- link link3_3: mass 0.202651 -> 0.150350

Commit message: Add files via upload

File: src/sim/urdf/robot.urdf (robot description, URDF)
Before this commit: robot my_robot_with_cage, 22 links, 21 joints
Links:
- link joint1: mass 0.431305 -> 0.639808643
- link link1_3: mass 0.322751 -> 0.450128794
- link link2_1: mass 0.840115 -> 0.697756362
