Commit message: urdf 수정

File: src/sim/urdf/robot.urdf (robot description, URDF)
Before this commit: robot my_robot_with_cage, 22 links, 21 joints
Links:
- link link2_1: mass 0.697756362 -> 0.41732128

Commit message: good_demo

File: src/sim/urdf/robot.urdf (robot description, URDF)
Before this commit: robot my_robot_with_cage, 22 links, 21 joints
Links:
- link joint1: mass 0.431305 -> 0.639808643
- link link1_3: mass 0.322751 -> 0.450128794
- link link2_1: mass 0.840115 -> 0.41732128
